File: eagle/rld-node.sch (EAGLE design)
At the start: 0 parts

Commit message: Added power supply
Parts:
- added C1, C2, C3, C4, C5, C6: (no value), rcl:C-EUC0805
- added R1, R2: (no value), rcl:R-EU_R0805
- added U$1, U$2: TPS6214X, texas-instruments:TPS6214X
- added X1: (no value), con-wago-500:W237-102
Connections:
- new net +3V3: C6.2, R2.2, U$2.VOS
- new net +5V: C3.2, R1.2, U$1.VOS
- new net GND: C1.2, C2.1, C3.1, C4.2, C5.1, C6.1, U$1.AGND, U$1.DEV, U$1.FB, U$1.FSW, U$1.PGND, U$2.AGND, U$2.DEV, U$2.FB, U$2.FSW, U$2.PGND, X1-2.KL
- new net N$1: C1.1, U$1.SS/TR
- new net N$2: C4.1, U$2.SS/TR
- new net N$3: R2.1, U$2.PG
- new net N$4: R1.1, U$1.PG
- new net VCC: C2.2, C5.2, U$1.AVIN, U$1.EN, U$1.PVIN, U$2.AVIN, U$2.EN, U$2.PVIN, X1-1.KL
